Commit message: Updated xacros and added gazebo_control. launch_sim.launch.py was added and relevent parmaters were added to then run on gazebo

File: description/robot.urdf.xacro (robot description, xacro)
@@ -2,3 +2,4 @@
 <robot xmlns:xacro="http://www.ros.org/wiki/xacro"  name="robot">
     <xacro:include filename="robot_core.xacro" />
+    <xacro:include filename="gazebo_control.xacro" />
 </robot>

File: description/robot_core.xacro (robot description, xacro)
@@ -41,4 +41,7 @@
         </xacro:inertial_box>
     </link>
+    <gazebo reference="chassis">
+        <material>Gazebo/White</material>
+    </gazebo>
     <!-- LEFT WHEEL LINK-->
     <joint name="left_wheel_joint" type="continuous">
@@ -60,8 +63,11 @@
             </geometry>
         </collision>
-        <xacro:inertial_cylinder mass="0.1" lenght="0.04" radius="0.05">
+        <xacro:inertial_cylinder mass="0.1" length="0.04" radius="0.05">
             <origin xyz="0 0 0" rpy="0 0 0"/>
         </xacro:inertial_cylinder>
     </link>
+    <gazebo reference="left_wheel">
+        <material>Gazebo/Blue</material>
+    </gazebo>
     <!-- RIGHT WHEEL LINK-->
     <joint name="right_wheel_joint" type="continuous">
@@ -83,8 +89,11 @@
             </geometry>
         </collision>
-        <xacro:inertial_cylinder mass="0.1" lenght="0.04" radius="0.05">
+        <xacro:inertial_cylinder mass="0.1" length="0.04" radius="0.05">
             <origin xyz="0 0 0" rpy="0 0 0"/>
         </xacro:inertial_cylinder>
     </link>
+    <gazebo reference="right_wheel">
+        <material>Gazebo/Blue</material>
+    </gazebo>
     <!-- CASTER WHEEL-->
     <joint name="caster_wheel_joint" type="fixed">
@@ -109,3 +118,8 @@
         </xacro:inertial_sphere>
     </link>
+    <gazebo reference="caster_wheel">
+        <material>Gazebo/Black</material>
+        <mu1 value="0.001"/>
+        <mu2 value="0.001"/>
+    </gazebo>
 </robot>

Commit message: Progress made -Working motors, working lidar, next step ros2 control

File: description/robot.urdf.xacro (robot description, xacro)
@@ -2,4 +2,6 @@
 <robot xmlns:xacro="http://www.ros.org/wiki/xacro"  name="robot">
     <xacro:include filename="robot_core.xacro" />
-    <xacro:include filename="gazebo_control.xacro" />
+    <!--<xacro:include filename="gazebo_control.xacro" /> -->
+    <xacro:include filename="ros2_control.xacro" />
+    <xacro:include filename="lidar.xacro" />
 </robot>

File: description/robot_core.xacro (robot description, xacro)
@@ -13,4 +13,7 @@
     <material name="black">
         <color rgba="0 0 0 1" />
+    </material>
+    <material name="red">
+        <color rgba="1 0 0 1" />
     </material>
     <!--BASE LINK -->

Commit message: Just general update on files

File: description/robot.urdf.xacro (robot description, xacro)
@@ -1,5 +1,12 @@
 <?xml version="1.0"?>
 <robot xmlns:xacro="http://www.ros.org/wiki/xacro"  name="robot">
+    <xacro:arg name="use_ros2_control" default="true"/>
     <xacro:include filename="robot_core.xacro" />
+    <xacro:if value="$(arg use_ros2_control)">
+        <xacro:include filename="ros2_control.xacro" />
+    </xacro:if>
+    <xacro:unless value="$(arg use_ros2_control)">
+        <xacro:include filename="gazebo_control.xacro" />
+    </xacro:unless>
     <!--<xacro:include filename="gazebo_control.xacro" /> -->
     <xacro:include filename="ros2_control.xacro" />

File: description/ros2_control.xacro (robot description, xacro)
@@ -1,5 +1,33 @@
 <?xml version="1.0"?>
 <robot xmlns:xacro="http://www.ros.org/wiki/xacro"  >
-    <ros2_control name="GazeboSystem" type="system">
+    <ros2_control name="RealRobot" type="system">
+        <hardware>
+            <plugin>diffdrive_arduino/DiffDriveArduino</plugin>
+            <param name="left_wheel_name">left_wheel_joint</param>
+            <param name="right_wheel_name">right_wheel_joint</param>
+            <param name="loop_rate">30</param>
+            <param name="device">/dev/ttyUSB0</param>
+            <param name="baud_rate">57600</param>
+            <param name="timeout">1000</param>
+            <param name="enc_counts_per_rev">3450</param>
+        </hardware>
+        <joint name="left_wheel_joint">
+            <command_interface name="velocity">
+                <param name="min">-10</param>
+                <param name="max">10</param>
+            </command_interface>
+            <state_interface name="velocity"/>
+            <state_interface name="position"/>
+        </joint>
+        <joint name="right_wheel_joint">
+            <command_interface name="velocity">
+                <param name="min">-10</param>
+                <param name="max">10</param>
+            </command_interface>
+            <state_interface name="velocity"/>
+            <state_interface name="position"/>
+        </joint>
+    </ros2_control>
+    <!-- <ros2_control name="GazeboSystem" type="system">
         <hardware>
             <plugin>gazebo_ros2_control/GazeboSystem</plugin>
@@ -21,5 +49,5 @@
             <state_interface name="position"/>
         </joint>
-    </ros2_control>
+    </ros2_control>-->
     <gazebo>
         <plugin name="gazebo_ros2_control" filename="libgazebo_ros2_control.so">
